Commit message: cleanup

File: giraffe_ws/src/giraffe_description/urdf/giraffe.urdf.xacro (robot description, xacro)
@@ -136,4 +136,5 @@
         <visual name="base_link_visual">
             <origin xyz="0.0 0.0 0.0" rpy="0.0 0.0 0.0" />
+            <material name="white"/>
             <geometry>
                 <mesh filename="package://giraffe_description/meshes/base_link.stl" scale="0.001 0.001 0.001" />
@@ -142,5 +143,4 @@
         <collision name="base_link_collision">
             <origin xyz="0.0 0.0 0.0" rpy="0.0 0.0 0.0" />
-            <material name="white"/>
             <geometry>
                 <mesh filename="package://giraffe_description/meshes/base_link.stl" scale="0.001 0.001 0.001" />
