Commit message: hardware and gazebo sim funct with moveit

File: giraffe_ws/src/giraffe_description/urdf/giraffe_ros2_control.xacro (robot description, xacro)
@@ -12,4 +12,10 @@
                 <plugin>gazebo_ros2_control/GazeboSystem</plugin>
             </hardware>
+            <!-- <hardware>
+                <plugin>topic_based_ros2_control/TopicBasedSystem</plugin>
+                <param name="joint_commands_topic">/topic_based_joint_commands</param>
+                <param name="joint_states_topic">/topic_based_joint_states</param>
+                <param name="sum_wrapped_joint_states">true</param>
+            </hardware> -->
             <joint name="base_link_shoulder_pan_joint">
                 <command_interface name="position">
@@ -18,7 +24,4 @@
                 </command_interface>
                 <state_interface name="position">
-                    <param name="initial_value">0.0</param>
-                </state_interface>
-                <state_interface name="velocity">
                     <param name="initial_value">0.0</param>
                 </state_interface>
@@ -32,7 +35,4 @@
                     <param name="initial_value">0.0</param>
                 </state_interface>
-                <state_interface name="velocity">
-                    <param name="initial_value">0.0</param>
-                </state_interface>
             </joint>
             <joint name="shoulder_lift_elbow_joint">
@@ -42,7 +42,4 @@
                 </command_interface>
                 <state_interface name="position">
-                    <param name="initial_value">0.0</param>
-                </state_interface>
-                <state_interface name="velocity">
                     <param name="initial_value">0.0</param>
                 </state_interface>
@@ -56,7 +53,4 @@
                     <param name="initial_value">0.0</param>
                 </state_interface>
-                <state_interface name="velocity">
-                    <param name="initial_value">0.0</param>
-                </state_interface>
             </joint>
             <joint name="wrist_1_wrist_2_joint">
@@ -66,7 +60,4 @@
                 </command_interface>
                 <state_interface name="position">
-                    <param name="initial_value">0.0</param>
-                </state_interface>
-                <state_interface name="velocity">
                     <param name="initial_value">0.0</param>
                 </state_interface>
@@ -80,7 +71,4 @@
                     <param name="initial_value">0.0</param>
                 </state_interface>
-                <state_interface name="velocity">
-                    <param name="initial_value">0.0</param>
-                </state_interface>
             </joint>
         </ros2_control>

File: giraffe_ws/src/giraffe_moveit_config/config/giraffe.ros2_control.xacro (robot description, xacro)
@@ -1,52 +1,74 @@
-<?xml version="1.0"?>
-<robot xmlns:xacro="http://www.ros.org/wiki/xacro">
-    <xacro:macro name="giraffe_ros2_control" params="name initial_positions_file">
-        <xacro:property name="initial_positions" value="${load_yaml(initial_positions_file)['initial_positions']}"/>
-        <ros2_control name="${name}" type="system">
+<?xml version="1.0" ?>
+<robot name="giraffe" xmlns:xacro="http://www.ros.org/wiki/xacro" >
+    <xacro:macro name="giraffe_ros2_control">
+        <gazebo>
+            <plugin filename="libgazebo_ros2_control.so" name="gazebo_ros2_control">
+                <robot_sim_type>gazebo_ros2_control/GazeboSystem</robot_sim_type>
+                <parameters>$(find giraffe_description)/config/giraffe_controller.yaml</parameters>
+            </plugin>
+        </gazebo>
+        <ros2_control name="GazeboSystem" type="system">
             <hardware>
-                <!-- By default, set up controllers for simulation. This won't work on real hardware -->
-                <plugin>mock_components/GenericSystem</plugin>
+                <plugin>giraffe_control/GiraffeHardwareInterface</plugin>
             </hardware>
+            <!-- <hardware>
+                <plugin>topic_based_ros2_control/TopicBasedSystem</plugin>
+                <param name="joint_commands_topic">/topic_based_joint_commands</param>
+                <param name="joint_states_topic">/topic_based_joint_states</param>
+                <param name="sum_wrapped_joint_states">true</param>
+            </hardware> -->
             <joint name="base_link_shoulder_pan_joint">
-                <command_interface name="position"/>
+                <command_interface name="position">
+                    <param name="min">-1.833</param>
+                    <param name="max">1.833</param>
+                </command_interface>
                 <state_interface name="position">
-                  <param name="initial_value">${initial_positions['base_link_shoulder_pan_joint']}</param>
+                    <param name="initial_value">0.0</param>
                 </state_interface>
-                <state_interface name="velocity"/>
             </joint>
             <joint name="shoulder_pan_shoulder_lift_joint">
-                <command_interface name="position"/>
+                <command_interface name="position">
+                    <param name="min">-0.785</param>
+                    <param name="max">1.644</param>
+                </command_interface>
                 <state_interface name="position">
-                  <param name="initial_value">${initial_positions['shoulder_pan_shoulder_lift_joint']}</param>
+                    <param name="initial_value">0.0</param>
                 </state_interface>
-                <state_interface name="velocity"/>
             </joint>
             <joint name="shoulder_lift_elbow_joint">
-                <command_interface name="position"/>
+                <command_interface name="position">
+                    <param name="min">-1.536</param>
+                    <param name="max">1.745</param>
+                </command_interface>
                 <state_interface name="position">
-                  <param name="initial_value">${initial_positions['shoulder_lift_elbow_joint']}</param>
+                    <param name="initial_value">0.0</param>
                 </state_interface>
-                <state_interface name="velocity"/>
             </joint>
             <joint name="elbow_wrist_1_joint">
-                <command_interface name="position"/>
+                <command_interface name="position">
+                    <param name="min">-3.368</param>
+                    <param name="max">0.262</param>
+                </command_interface>
                 <state_interface name="position">
-                  <param name="initial_value">${initial_positions['elbow_wrist_1_joint']}</param>
+                    <param name="initial_value">0.0</param>
                 </state_interface>
-                <state_interface name="velocity"/>
             </joint>
             <joint name="wrist_1_wrist_2_joint">
-                <command_interface name="position"/>
+                <command_interface name="position">
+                    <param name="min">-3.142</param>
+                    <param name="max">3.142</param>
+                </command_interface>
                 <state_interface name="position">
-                  <param name="initial_value">${initial_positions['wrist_1_wrist_2_joint']}</param>
+                    <param name="initial_value">0.0</param>
                 </state_interface>
-                <state_interface name="velocity"/>
             </joint>
             <joint name="wrist_2_gripper_joint">
-                <command_interface name="position"/>
+                <command_interface name="position">
+                    <param name="min">-0.175</param>
+                    <param name="max">1.571</param>
+                </command_interface>
                 <state_interface name="position">
-                  <param name="initial_value">${initial_positions['wrist_2_gripper_joint']}</param>
+                    <param name="initial_value">0.0</param>
                 </state_interface>
-                <state_interface name="velocity"/>
             </joint>
         </ros2_control>

File: giraffe_ws/src/giraffe_moveit_config/config/giraffe.urdf.xacro (robot description, xacro)
@@ -6,4 +6,4 @@
     <!-- Import control_xacro -->
     <xacro:include filename="giraffe.ros2_control.xacro" />
-    <xacro:giraffe_ros2_control name="FakeSystem" initial_positions_file="$(arg initial_positions_file)"/>
+    <xacro:giraffe_ros2_control/>
 </robot>
